Commit message: urdf rviz

File: kinova_description/urdf/jaco_arm_cylinder.urdf (robot description, URDF)
Before this commit: robot jaco_arm, 10 links, 9 joints
Links:
- removed link j2n6s300_end_effector
- added link ee_cylinder, mass 0.1; collision cylinder length=0.08 radius=0.02; visual cylinder length=0.08 radius=0.02
Joints:
- removed joint j2n6s300_joint_end_effector
- added joint joint_end_effector2: type fixed, parent j2n6s300_link_6, child ee_cylinder, origin xyz=0 0 -0.081 rpy=0 0 0, axis 0 0 0

Commit message: cleanup

File: kinova_description/urdf/jaco_arm_cylinder.urdf (robot description, URDF)
Before this commit: robot jaco_arm, 10 links, 9 joints
Joints:
- joint joint_end_effector2: origin xyz=0 0 -0.081 rpy=0 0 0 -> xyz=0 0 -0.041 rpy=0 0 0

Commit message: more debugging of actions and state

File: kinova_description/urdf/jaco_arm_cylinder.urdf (robot description, URDF)
Before this commit: robot jaco_arm, 10 links, 9 joints
Joints:
- joint joint_end_effector2: origin xyz=0 0 -0.041 rpy=0 0 0 -> xyz=0 0 -0.04 rpy=0 0 0
